File: AngularRGB.kicad_pcb (KiCad board)
At the start: 4 copper layers, 228.6 x 76.2 mm, 192 parts, among them Q1 BSS138, SW1 SW_Push, SW1.25U1 MX_1.25U, SW1.25U2 MX_1.25U, SW1.25U3 MX_1.25U, SW1.25U4 MX_1.25U, SW1.25U5 MX_1.25U, SW1.25U6 MX_1.25U, SW1.75U1 MX_1.75U, SW1.75U2 MX_1.75U, SW10 MX_1U, SW11 MX_1U, SW12 MX_1U, SW13 MX_1U, SW14 MX_1U, SW15 MX_1U, SW16 MX_1U, SW17 MX_1U, SW18 MX_1U, SW19 MX_1U, SW2 MX_1U, SW2.25U1 MX_2.25U, SW2.75U1 MX_2.75U, SW20 MX_1U, SW21 MX_1U, SW22 MX_1U, SW23 MX_1U, SW24 MX_1U, SW25 MX_1U, SW26 MX_1U, SW27 MX_1U, SW28 MX_1U, SW29 MX_1U, SW3 MX_1U, SW30 MX_1U, SW31 MX_1U, SW32 MX_1U, SW33 MX_1U, SW4 MX_1U, SW5 MX_1U, SW6 MX_1U, SW7 MX_1U, SW8 MX_1U, SW9 MX_1U, U1 ATmega32U4-MU, U2 USB6B1, U3 74LVC2G34, U4 AMS1117-3.3, U5 nRF51x22-QFxx, Y1 Crystal_GND24, Y2 Crystal_GND24

Commit message: First commit
Parts:
- removed F1: Fuse, Fuse:Fuse_0603_1608Metric
- added C30: 10uF, Capacitor_SMD:C_0805_2012Metric, B.Cu at (194.0, 114.7)
- added C31: 1uF, Capacitor_SMD:C_0603_1608Metric, B.Cu at (155.3, 121.2)
- added C32: 100n, Capacitor_SMD:C_0603_1608Metric, B.Cu at (162.8, 117.7)
- added C33: 10uF, Capacitor_SMD:C_0805_2012Metric, B.Cu at (149.9, 117.9)
- added C34: 10uF, Capacitor_SMD:C_0805_2012Metric, B.Cu at (138.4, 121.2)
- added D44: LED, LED_SMD:LED_0603_1608Metric, B.Cu at (194.6, 117.9)
- added D45: LED, LED_SMD:LED_0603_1608Metric, B.Cu at (193.0, 117.9)
- added D46: D_Schottky, Diode_SMD:D_SMB, B.Cu at (143.5, 122.2)
- added D47: D_Schottky, Diode_SMD:D_SMB, B.Cu at (118.1, 118.4)
- added D48: D_Schottky, Diode_SMD:D_SMB, B.Cu at (118.1, 122.6)
- added L4: 10uH, Inductor_SMD:L_0805_2012Metric, B.Cu at (149.0, 120.9)
- added Q2: 2N7000, Package_TO_SOT_SMD:SOT-23, B.Cu at (158.2, 121.4)
- added Q3: 2N7000, Package_TO_SOT_SMD:SOT-23, B.Cu at (161.8, 121.4)
- added R10: 1k, Resistor_SMD:R_0603_1608Metric, B.Cu at (193.8, 120.1)
- added R11: 1k, Resistor_SMD:R_0603_1608Metric, B.Cu at (193.8, 121.7)
- added R12: 2k, Resistor_SMD:R_0603_1608Metric, B.Cu at (197.9, 114.6)
- added R13: 100, Resistor_SMD:R_0603_1608Metric, B.Cu at (156.7, 115.1)
- added R14: 2k, Resistor_SMD:R_0603_1608Metric, B.Cu at (155.3, 117.7)
- added R15: 7.5k, Resistor_SMD:R_0603_1608Metric, B.Cu at (143.3, 117.0)
- added R16: 1k, Resistor_SMD:R_0603_1608Metric, B.Cu at (143.4, 118.5)
- added SW34: SW_DIP_x01, Button_Switch_SMD:SW_DIP_SPSTx01_Slide_6.7x4.1mm_W6.73mm_P2.54mm_LowProfile_JPin, F.Cu at (152.8, 126.7)
- added TP3: B+, TestPoint:TestPoint_Pad_D3.0mm, B.Cu at (198.5, 126.0)
- added TP4: B-, TestPoint:TestPoint_Pad_D3.0mm, B.Cu at (193.7, 126.0)
- added TP5: TestPoint, TestPoint:TestPoint_Pad_D2.0mm, B.Cu at (120.1, 126.7)
- added U6: TP4056, Package_SO:MSOP-8-1EP_3x3mm_P0.65mm_EP2.54x2.8mm, B.Cu at (197.9, 119.1)
- added U7: FS312F, Package_TO_SOT_SMD:SOT-23-6, B.Cu at (159.6, 117.8)
- added U8: MT3608, Package_TO_SOT_SMD:SOT-23-6, B.Cu at (146.9, 118.0)
- C27, C29: moved to B.Cu
- D1: footprint Diode_SMD:D_SOD-123F -> Diode_SMD:D_SOD-123
- TP1, TP2: moved to F.Cu
- moved C6 92.5 mm to (110.3, 123.4), turned to 90 degrees
- moved C4 91.3 mm to (110.4, 120.2), turned to 90 degrees
- moved C3 89.0 mm to (107.1, 126.3), turned to 90 degrees
- moved C5 88.8 mm to (110.4, 116.9), turned to 90 degrees
- moved Y1 86.5 mm to (104.0, 126.3), turned to 0 degrees
- moved C2 86.2 mm to (101.0, 126.4), turned to 270 degrees
- moved C1 85.6 mm to (100.6, 112.8), turned to 0 degrees
- moved C7 81.9 mm to (107.4, 112.8), turned to 180 degrees
- moved U1 81.0 mm to (104.0, 119.0), turned to 180 degrees
- moved D43 79.5 mm to (317.9, 75.5)
- moved U4 79.5 mm to (311.6, 67.0)
- moved U3 79.5 mm to (313.0, 74.9)
- moved C8 77.3 mm to (97.8, 121.9), turned to 270 degrees
- moved C20 77.0 mm to (312.5, 59.2)
- moved C17 77.0 mm to (302.5, 59.7)
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Connections:
- net /VBUS renamed VBUS
Routing:
- net R0: track 0.00 -> 209.5 mm
- net R2: track 0.00 -> 208.6 mm
- net R3: track 0.00 -> 207.4 mm
- net R1: track 0.00 -> 200.0 mm
- net VBUS: track 0.00 -> 120.0 mm, vias 0 -> 8
- net /BAT+: track 0.00 -> 66.4 mm, vias 0 -> 4
- net /D+: track 0.00 -> 66.3 mm, vias 0 -> 2
- net /D-: track 0.00 -> 65.1 mm, vias 0 -> 2
- net Net-(D4-Pad2): track 0.00 -> 47.3 mm
- net Net-(D34-Pad2): track 0.00 -> 45.9 mm
- net /BAT-: track 0.00 -> 42.9 mm
- net Net-(D41-Pad2): track 0.00 -> 42.5 mm
- net Net-(D27-Pad2): track 0.00 -> 42.3 mm
- net Net-(D11-Pad2): track 0.00 -> 41.7 mm
- net Net-(D7-Pad2): track 0.00 -> 38.9 mm
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Other:
- board text added: "+"
- board text added: "-"
- board text added: "VBAT"
