File: AngularRGB.sch (KiCad schematic (older format))
At the start: 217 parts, among them Q1 BSS138, Q2 2N7000, Q3 2N7000, SW1 SW_Push, SW1.25U1 MX_1.25U, SW1.25U2 MX_1.25U, SW1.25U3 MX_1.25U, SW1.25U4 MX_1.25U, SW1.25U5 MX_1.25U, SW1.25U6 MX_1.25U, SW1.75U1 MX_1.75U, SW1.75U2 MX_1.75U, SW10 MX_1U, SW11 MX_1U, SW12 MX_1U, SW13 MX_1U, SW14 MX_1U, SW15 MX_1U, SW16 MX_1U, SW17 MX_1U, SW18 MX_1U, SW19 MX_1U, SW2 MX_1U, SW2.25U1 MX_2.25U, SW2.75U1 MX_2.75U, SW20 MX_1U, SW21 MX_1U, SW22 MX_1U, SW23 MX_1U, SW24 MX_1U, SW25 MX_1U, SW26 MX_1U, SW27 MX_1U, SW28 MX_1U, SW29 MX_1U, SW3 MX_1U, SW30 MX_1U, SW31 MX_1U, SW32 MX_1U, SW33 MX_1U, SW34 SW_DIP_x01, SW4 MX_1U, SW5 MX_1U, SW6 MX_1U, SW7 MX_1U, SW8 MX_1U, SW9 MX_1U, U1 ATmega32U4-MU, U2 USB6B1, U3 74LVC2G34, U4 AMS1117-3.3, U5 nRF51x22-QFxx, U6 TP4056, U7 FS312F, U8 MT3608, Y1 Crystal_GND24, Y2 Crystal_GND24

Commit message: First commit
Parts:
- added TP5: TestPoint, TestPoint:TestPoint_Pad_D2.0mm, symbol Connector:TestPoint
- C30, C33, C34: footprint (none) -> Capacitor_SMD:C_0805_2012Metric
- C31, C32: footprint (none) -> Capacitor_SMD:C_0603_1608Metric
- D1: footprint Diode_SMD:D_SOD-123F -> Diode_SMD:D_SOD-123
- D44, D45: footprint (none) -> LED_SMD:LED_0603_1608Metric
- D46, D47, D48: footprint (none) -> Diode_SMD:D_SMB
- L4: footprint (none) -> Inductor_SMD:L_0805_2012Metric
- Q2, Q3: footprint Package_TO_SOT_THT:TO-92_Inline -> Package_TO_SOT_SMD:SOT-23
- R10, R11, R12, R13, R14, R15, R16: footprint (none) -> Resistor_SMD:R_0603_1608Metric
- SW34: footprint (none) -> Button_Switch_SMD:SW_DIP_SPSTx01_Slide_6.7x4.1mm_W6.73mm_P2.54mm_LowProfile_JPin
- TP3, TP4: footprint (none) -> TestPoint:TestPoint_Pad_D3.0mm
- U6: footprint (none) -> Package_SO:MSOP-8-1EP_3x3mm_P0.65mm_EP2.54x2.8mm
- U7, U8: footprint (none) -> Package_TO_SOT_SMD:SOT-23-6
Connections:
- net labels added: PPBUS_HOT
- wire segments 858 -> 857
Other:
- moved on the sheet: D47, D48
Changed lines of the file:
@@
 F 0 "D1" H 5750 3676 50  0000 C CNN
 F 1 "D" H 5750 3675 50  0001 C CNN
-F 2 "Diode_SMD:D_SOD-123F" H 5750 3800 50  0001 C CNN
+F 2 "Diode_SMD:D_SOD-123" H 5750 3800 50  0001 C CNN
 F 3 "~" H 5750 3800 50  0001 C CNN
 	1    5750 3800
@@
 F 0 "U6" H 5250 8700 50  0000 C CNN
 F 1 "TP4056" H 5250 8000 50  0000 C CNN
-F 2 "" H 5250 8400 50  0001 C CNN
+F 2 "Package_SO:MSOP-8-1EP_3x3mm_P0.65mm_EP2.54x2.8mm" H 5250 8400 50  0001 C CNN
 F 3 "" H 5250 8400 50  0001 C CNN
 	1    5250 8400
@@
 F 0 "C30" H 4065 8346 50  0000 L CNN
 F 1 "10uF" H 4065 8255 50  0000 L CNN
-F 2 "" H 3988 8150 50  0001 C CNN
+F 2 "Capacitor_SMD:C_0805_2012Metric" H 3988 8150 50  0001 C CNN
 F 3 "~" H 3950 8300 50  0001 C CNN
 	1    3950 8300
@@
 F 0 "D44" V 4288 8383 50  0000 R CNN
 F 1 "LED" V 4197 8383 50  0000 R CNN
-F 2 "" H 4250 8500 50  0001 C CNN
+F 2 "LED_SMD:LED_0603_1608Metric" H 4250 8500 50  0001 C CNN
 F 3 "~" H 4250 8500 50  0001 C CNN
 	1    4250 8500
@@
 F 0 "D45" V 4638 8383 50  0000 R CNN
 F 1 "LED" V 4547 8383 50  0000 R CNN
-F 2 "" H 4600 8500 50  0001 C CNN
+F 2 "LED_SMD:LED_0603_1608Metric" H 4600 8500 50  0001 C CNN
 F 3 "~" H 4600 8500 50  0001 C CNN
 	1    4600 8500
@@
 F 0 "TP3" V 6254 8438 50  0000 L CNN
 F 1 "B+" V 6345 8438 50  0000 L CNN
-F 2 "" H 6500 8250 50  0001 C CNN
+F 2 "TestPoint:TestPoint_Pad_D3.0mm" H 6500 8250 50  0001 C CNN
 F 3 "~" H 6500 8250 50  0001 C CNN
 	1    6300 8250
@@
 F 0 "TP4" V 8004 8738 50  0000 L CNN
 F 1 "B-" V 8095 8738 50  0000 L CNN
-F 2 "" H 8250 8550 50  0001 C CNN
+F 2 "TestPoint:TestPoint_Pad_D3.0mm" H 8250 8550 50  0001 C CNN
 F 3 "~" H 8250 8550 50  0001 C CNN
 	1    8050 8550
@@
 F 0 "R11" H 4670 8846 50  0000 L CNN
 F 1 "1k" H 4670 8755 50  0000 L CNN
-F 2 "" V 4530 8800 50  0001 C CNN
+F 2 "Resistor_SMD:R_0603_1608Metric" V 4530 8800 50  0001 C CNN
 F 3 "~" H 4600 8800 50  0001 C CNN
 	1    4600 8800
@@
 F 0 "R10" H 4320 8846 50  0000 L CNN
 F 1 "1k" H 4320 8755 50  0000 L CNN
-F 2 "" V 4180 8800 50  0001 C CNN
+F 2 "Resistor_SMD:R_0603_1608Metric" V 4180 8800 50  0001 C CNN
 F 3 "~" H 4250 8800 50  0001 C CNN
 	1    4250 8800
@@
 F 0 "C31" H 5865 8996 50  0000 L CNN
 F 1 "1uF" H 5865 8905 50  0000 L CNN
-F 2 "" H 5788 8800 50  0001 C CNN
+F 2 "Capacitor_SMD:C_0603_1608Metric" H 5788 8800 50  0001 C CNN
 F 3 "~" H 5750 8950 50  0001 C CNN
 	1    5750 8950
@@
 F 0 "R12" H 6170 8996 50  0000 L CNN
 F 1 "2k" H 6170 8905 50  0000 L CNN
-F 2 "" V 6030 8950 50  0001 C CNN
+F 2 "Resistor_SMD:R_0603_1608Metric" V 6030 8950 50  0001 C CNN
 F 3 "~" H 6100 8950 50  0001 C CNN
 	1    6100 8950
@@
 F 0 "U7" H 7400 8700 50  0000 C CNN
 F 1 "FS312F" H 7400 8200 50  0000 C CNN
-F 2 "" H 7400 8400 50  0001 C CNN
+F 2 "Package_TO_SOT_SMD:SOT-23-6" H 7400 8400 50  0001 C CNN
 F 3 "" H 7400 8400 50  0001 C CNN
 	1    7400 8400
@@
 F 0 "Q2" V 7350 9000 50  0000 C CNN
 F 1 "2N7000" V 7441 9000 50  0000 C CNN
-F 2 "Package_TO_SOT_THT:TO-92_Inline" H 7300 8925 50  0001 L CIN
+F 2 "Package_TO_SOT_SMD:SOT-23" H 7300 8925 50  0001 L CIN
 F 3 "https://www.fairchildsemi.com/datasheets/2N/2N7000.pdf" H 7100 9000 50  0001 L CNN
 	1    7100 9000
@@
 F 0 "Q3" V 8043 9200 50  0000 C CNN
 F 1 "2N7000" V 7952 9200 50  0000 C CNN
-F 2 "Package_TO_SOT_THT:TO-92_Inline" H 7900 9125 50  0001 L CIN
+F 2 "Package_TO_SOT_SMD:SOT-23" H 7900 9125 50  0001 L CIN
 F 3 "https://www.fairchildsemi.com/datasheets/2N/2N7000.pdf" H 7700 9200 50  0001 L CNN
 	1    7700 9200
@@
 F 0 "R14" H 6870 8696 50  0000 L CNN
 F 1 "2k" H 6870 8605 50  0000 L CNN
-F 2 "" V 6730 8650 50  0001 C CNN
+F 2 "Resistor_SMD:R_0603_1608Metric" V 6730 8650 50  0001 C CNN
 F 3 "~" H 6800 8650 50  0001 C CNN
 	1    6800 8650
@@
 F 0 "C32" H 8165 8196 50  0000 L CNN
 F 1 "100n" H 8165 8105 50  0000 L CNN
-F 2 "" H 8088 8000 50  0001 C CNN
+F 2 "Capacitor_SMD:C_0603_1608Metric" H 8088 8000 50  0001 C CNN
 F 3 "~" H 8050 8150 50  0001 C CNN
 	1    8050 8150
@@
 F 0 "R13" V 6343 8000 50  0000 C CNN
 F 1 "100" V 6434 8000 50  0000 C CNN
-F 2 "" V 6480 8000 50  0001 C CNN
+F 2 "Resistor_SMD:R_0603_1608Metric" V 6480 8000 50  0001 C CNN
 F 3 "~" H 6550 8000 50  0001 C CNN
 	1    6550 8000
@@
 F 0 "U8" H 10250 8185 50  0000 C CNN
 F 1 "MT3608" H 10250 8276 50  0000 C CNN
-F 2 "" H 10250 8500 50  0001 C CNN
+F 2 "Package_TO_SOT_SMD:SOT-23-6" H 10250 8500 50  0001 C CNN
 F 3 "" H 10250 8500 50  0001 C CNN
 	1    10250 8500
@@
 F 0 "SW34" H 9100 8267 50  0000 C CNN
 F 1 "SW_DIP_x01" H 9100 8176 50  0000 C CNN
-F 2 "" H 9100 8000 50  0001 C CNN
+F 2 "Button_Switch_SMD:SW_DIP_SPSTx01_Slide_6.7x4.1mm_W6.73mm_P2.54mm_LowProfile_JPin" H 9100 8000 50  0001 C CNN
 F 3 "" H 9100 8000 50  0001 C CNN
 	1    9100 8000
@@
 F 0 "L4" V 10440 8000 50  0000 C CNN
 F 1 "10uH" V 10349 8000 50  0000 C CNN
-F 2 "" H 10250 8000 50  0001 C CNN
+F 2 "Inductor_SMD:L_0805_2012Metric" H 10250 8000 50  0001 C CNN
 F 3 "~" H 10250 8000 50  0001 C CNN
 	1    10250 8000
@@
 F 0 "D46" H 10850 7784 50  0000 C CNN
 F 1 "D_Schottky" H 10850 7875 50  0000 C CNN
-F 2 "" H 10850 8000 50  0001 C CNN
+F 2 "Diode_SMD:D_SMB" H 10850 8000 50  0001 C CNN
 F 3 "~" H 10850 8000 50  0001 C CNN
 	1    10850 8000
@@
 F 0 "R15" H 11120 8346 50  0000 L CNN
 F 1 "7.5k" H 11120 8255 50  0000 L CNN
-F 2 "" V 10980 8300 50  0001 C CNN
+F 2 "Resistor_SMD:R_0603_1608Metric" V 10980 8300 50  0001 C CNN
 F 3 "~" H 11050 8300 50  0001 C CNN
 	1    11050 8300
@@
 F 0 "R16" H 11120 8646 50  0000 L CNN
 F 1 "1k" H 11120 8555 50  0000 L CNN
-F 2 "" V 10980 8600 50  0001 C CNN
+F 2 "Resistor_SMD:R_0603_1608Metric" V 10980 8600 50  0001 C CNN
 F 3 "~" H 11050 8600 50  0001 C CNN
 	1    11050 8600
@@
 F 0 "C33" H 9765 8296 50  0000 L CNN
 F 1 "10uF" H 9765 8205 50  0000 L CNN
-F 2 "" H 9688 8100 50  0001 C CNN
+F 2 "Capacitor_SMD:C_0805_2012Metric" H 9688 8100 50  0001 C CNN
 F 3 "~" H 9650 8250 50  0001 C CNN
 	1    9650 8250
@@
 F 0 "C34" H 11565 8496 50  0000 L CNN
 F 1 "10uF" H 11565 8405 50  0000 L CNN
-F 2 "" H 11488 8300 50  0001 C CNN
+F 2 "Capacitor_SMD:C_0805_2012Metric" H 11488 8300 50  0001 C CNN
 F 3 "~" H 11450 8450 50  0001 C CNN
 	1    11450 8450
@@
 L Device:D_Schottky D47
 U 1 1 63AB98B0
-P 12400 8000
-F 0 "D47" H 12400 7784 50  0000 C CNN
-F 1 "D_Schottky" H 12400 7875 50  0000 C CNN
-F 2 "" H 12400 8000 50  0001 C CNN
-F 3 "~" H 12400 8000 50  0001 C CNN
-	1    12400 8000
+P 13300 8000
+F 0 "D47" H 13300 7784 50  0000 C CNN
+F 1 "D_Schottky" H 13300 7875 50  0000 C CNN
+F 2 "Diode_SMD:D_SMB" H 13300 8000 50  0001 C CNN
+F 3 "~" H 13300 8000 50  0001 C CNN
+	1    13300 8000
 	-1   0    0    1
 $EndComp
@@
 L Device:D_Schottky D48
 U 1 1 63ABA10C
-P 12400 8400
-F 0 "D48" H 12400 8184 50  0000 C CNN
-F 1 "D_Schottky" H 12400 8275 50  0000 C CNN
-F 2 "" H 12400 8400 50  0001 C CNN
-F 3 "~" H 12400 8400 50  0001 C CNN
-	1    12400 8400
+P 13300 8400
+F 0 "D48" H 13300 8184 50  0000 C CNN
+F 1 "D_Schottky" H 13300 8275 50  0000 C CNN
+F 2 "Diode_SMD:D_SMB" H 13300 8400 50  0001 C CNN
+F 3 "~" H 13300 8400 50  0001 C CNN
+	1    13300 8400
 	-1   0    0    1
 $EndComp
@@
 L power:VBUS #PWR048
 U 1 1 63B7A6E0
-P 12050 7900
-F 0 "#PWR048" H 12050 7750 50  0001 C CNN
-F 1 "VBUS" H 11900 7950 50  0000 C CNN
-F 2 "" H 12050 7900 50  0001 C CNN
-F 3 "" H 12050 7900 50  0001 C CNN
-	1    12050 7900
+P 12950 7900
+F 0 "#PWR048" H 12950 7750 50  0001 C CNN
+F 1 "VBUS" H 12800 7950 50  0000 C CNN
+F 2 "" H 12950 7900 50  0001 C CNN
+F 3 "" H 12950 7900 50  0001 C CNN
+	1    12950 7900
 	1    0    0    -1
 $EndComp
@@
 L power:+BATT #PWR049
 U 1 1 63B7A8D7
-P 12050 8300
-F 0 "#PWR049" H 12050 8150 50  0001 C CNN
-F 1 "+BATT" H 11900 8350 50  0000 C CNN
-F 2 "" H 12050 8300 50  0001 C CNN
-F 3 "" H 12050 8300 50  0001 C CNN
-	1    12050 8300
+P 12950 8300
+F 0 "#PWR049" H 12950 8150 50  0001 C CNN
+F 1 "+BATT" H 12800 8350 50  0000 C CNN
+F 2 "" H 12950 8300 50  0001 C CNN
+F 3 "" H 12950 8300 50  0001 C CNN
+	1    12950 8300
 	1    0    0    -1
 $EndComp
 Wire Wire Line
-	12050 8400 12250 8400
+	12950 8400 13150 8400
 Wire Wire Line
-	12050 8300 12050 8400
-$Comp
-L power:VCC #PWR050
-U 1 1 63E7F039
-P 13050 8100
-F 0 "#PWR050" H 13050 7950 50  0001 C CNN
-F 1 "VCC" H 13067 8273 50  0000 C CNN
-F 2 "" H 13050 8100 50  0001 C CNN
-F 3 "" H 13050 8100 50  0001 C CNN
-	1    13050 8100
-	1    0    0    -1
-$EndComp
-Wire Wire Line
-	12550 8400 12650 8400
+	12950 8300 12950 8400
 Wire Wire Line
-	12650 8400 12650 8200
+	13450 8400 13550 8400
 Wire Wire Line
-	12650 8000 12550 8000
+	13550 8400 13550 8200
 Wire Wire Line
-	12250 8000 12050 8000
+	13550 8000 13450 8000
 Wire Wire Line
-	12050 8000 12050 7900
+	13150 8000 12950 8000
 Wire Wire Line
-	12650 8200 13050 8200
-Connection ~ 12650 8200
+	12950 8000 12950 7900
+Connection ~ 13550 8200
 Wire Wire Line
-	12650 8200 12650 8000
-Wire Wire Line
-	13050 8100 13050 8200
+	13550 8200 13550 8000
 Wire Wire Line
 	4900 8550 4850 8550
@@
 Wire Wire Line
 	4850 8950 4600 8950
+Wire Wire Line
+	13550 8200 14100 8200
+Text Label 13650 8200 0    50   ~ 0
+PPBUS_HOT
+$Comp
+L Connector:TestPoint TP5
+U 1 1 5D15EBE1
+P 11450 8000
+F 0 "TP5" V 11404 8188 50  0000 L CNN
+F 1 "TestPoint" V 11495 8188 50  0000 L CNN
+F 2 "TestPoint:TestPoint_Pad_D2.0mm" H 11650 8000 50  0001 C CNN
+F 3 "~" H 11650 8000 50  0001 C CNN
+	1    11450 8000
+	0    1    1    0
+$EndComp
 $EndSCHEMATC
